File: device.sch (EAGLE design)
At the start: 48 parts, among them J0 S2B-PH-SM4-TB(LF)(SN), J1 JST_ZH_2PIN, J2 JST_ZH_2PIN, J3 JST_ZH_2PIN, J4 JST_ZH_2PIN, J5 JST_ZH_2PIN, J6 JST_ZH_2PIN, Q1 2SC2712-GR(F), Q2 2SC2712-GR(F), Q3 2SC2712-GR(F)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

Commit message: update files
Changed lines of the file:
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@@
 <attribute name="VALUE" x="71.12" y="17.78" size="1.778" layer="96"/>
 </instance>
-<instance part="GND11" gate="1" x="86.36" y="20.32" smashed="yes">
-<attribute name="VALUE" x="83.82" y="17.78" size="1.778" layer="96"/>
+<instance part="GND11" gate="1" x="86.36" y="38.1" smashed="yes">
+<attribute name="VALUE" x="83.82" y="35.56" size="1.778" layer="96"/>
 </instance>
 <instance part="GND12" gate="1" x="12.7" y="7.62" smashed="yes">
@@
 <pinref part="SV1" gate="G$1" pin="1"/>
 <wire x1="106.68" y1="50.8" x2="86.36" y2="50.8" width="0.1524" layer="91"/>
-<wire x1="86.36" y1="50.8" x2="86.36" y2="22.86" width="0.1524" layer="91"/>
+<wire x1="86.36" y1="50.8" x2="86.36" y2="40.64" width="0.1524" layer="91"/>
 <pinref part="GND11" gate="1" pin="GND"/>
 </segment>
@@
 <pinref part="J6" gate="G$1" pin="P$2"/>
 <wire x1="-134.62" y1="5.08" x2="-129.54" y2="5.08" width="0.1524" layer="91"/>
-</segment>
-<segment>
+<label x="-132.08" y="7.62" size="1.778" layer="95"/>
+</segment>
+<segment>
